File: keyboard.kicad_pcb (KiCad board)
At the start: 2 copper layers, 355.7 x 122.3 mm, 199 parts, among them J1 USB_B_Micro, J2 Conn_01x02, U1 NCP1117-3.3_SOT223, U2 W25Q128JVS, U3 RP2040, Y1 ABLS-12.000MHZ-B4-T

Commit message: add breakout, mini-DIN, and display headers; re-route
Parts:
- added C6: 100n, Capacitor_SMD:C_0402_1005Metric, F.Cu at (297.9, 2.41)
- added C7: 100n, Capacitor_SMD:C_0402_1005Metric, F.Cu at (296.5, 2.41)
- added C8: 1u, Capacitor_SMD:C_0402_1005Metric, B.Cu at (290.7, 3.17)
- added D88: 1N4148W, Diode_SMD:D_0402_1005Metric, F.Cu at (266.8, 5.71)
- added D89: 1N4148W, Diode_SMD:D_0402_1005Metric, B.Cu at (256.9, 8.64)
- added D90: 1N4148W, Diode_SMD:D_0402_1005Metric, F.Cu at (228.0, 6.35)
- added D91: 1N4148W, Diode_SMD:D_0402_1005Metric, F.Cu at (198.4, 8.51)
- added J3: Mini-DIN-6, RP2040_minimal:MJD-006-FS, F.Cu at (187.2, 8.89)
- added J4: Breakout, Connector_PinHeader_2.54mm:PinHeader_1x07_P2.54mm_Vertical, F.Cu at (209.4, 3.17)
- added J5: I2C_Display_Header, Connector_PinHeader_2.54mm:PinHeader_1x04_P2.54mm_Horizontal, F.Cu at (166.0, 13.7)
- C1, C10, C4, J1, R3, R4, R5, U1, U3: moved to F.Cu
- moved Y1 82.0 mm to (307.5, 9.78)
- moved C3 82.0 mm to (301.5, 13.1), turned to 180 degrees
- moved C2 81.9 mm to (310.5, 13.1), turned to 180 degrees
- moved C17 73.1 mm to (340.2, 7.37), turned to 180 degrees
- moved U3 73.1 mm to (291.8, 7.62)
- moved C10 69.2 mm to (297.8, 4.57), turned to 0 degrees
- moved C9 67.9 mm to (352.6, 12.9), turned to 90 degrees
- moved C11 66.5 mm to (350.3, 12.9), turned to 90 degrees
- moved R3 65.9 mm to (292.0, 2.03)
- moved R4 65.7 mm to (292.0, 0.89)
- moved C12 65.3 mm to (347.9, 12.9), turned to 90 degrees
- moved R2 64.7 mm to (329.9, 1.27)
- moved C13 64.5 mm to (345.6, 12.9), turned to 90 degrees
- moved C16 64.1 mm to (338.8, 12.9), turned to 90 degrees
- moved C14 64.0 mm to (343.3, 12.9), turned to 90 degrees
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Connections:
- J1 pad 1: VBUS -> Net-(D88-Pad2)
- U3 pad 11: col8 -> col6
- U3 pad 12: col9 -> col5
- U3 pad 13: /GPIO10 -> col4
- U3 pad 14: /GPIO11 -> col3
- U3 pad 15: /GPIO12 -> col2
- U3 pad 16: /GPIO13 -> col1
- U3 pad 17: /GPIO14 -> col0
- U3 pad 18: /GPIO15 -> col15
- U3 pad 2: col0 -> col9
- U3 pad 23: Net-(U3-Pad23) -> +1V1
- U3 pad 27: row3 -> col16
- U3 pad 28: col14 -> col17
- U3 pad 29: col13 -> row0
- U3 pad 3: col1 -> col10
- U3 pad 30: col12 -> row1
- U3 pad 31: col11 -> row2
- U3 pad 32: col10 -> row3
- U3 pad 34: row1 -> row4
- U3 pad 35: row0 -> row5
- U3 pad 36: col17 -> /GPIO24
- U3 pad 37: row2 -> /GPIO25
- U3 pad 38: row4 -> /GPIO26_ADC0
- U3 pad 39: col16 -> /GPIO27_ADC1
- U3 pad 4: col2 -> col11
- U3 pad 40: row5 -> /I2C_SDA
- U3 pad 41: col15 -> /I2C_SCL
- U3 pad 45: Net-(U3-Pad45) -> +1V1
- U3 pad 5: col3 -> col12
- U3 pad 50: Net-(U3-Pad50) -> +1V1
- U3 pad 6: col4 -> col13
- U3 pad 7: col5 -> col14
- U3 pad 8: col6 -> col8
Routing:
- net /I2C_SDA: track 0.00 -> 147.6 mm, vias 0 -> 2
- net /I2C_SCL: track 0.00 -> 145.1 mm, vias 0 -> 2
- net /GPIO25: track 0.00 -> 144.4 mm, vias 0 -> 2
- net /GPIO24: track 0.00 -> 143.3 mm, vias 0 -> 1
- net +3V3: track 46.8 -> 184.0 mm, vias 3 -> 2
- net /GPIO26_ADC0: track 0.00 -> 134.7 mm, vias 0 -> 2
- net /GPIO27_ADC1: track 0.00 -> 134.5 mm, vias 0 -> 1
- net GND: track 102.8 -> 233.7 mm, vias 10 -> 13
- net VBUS: track 16.6 -> 129.1 mm, vias 2 -> 5
- net col15: track 206.0 -> 117.0 mm, vias 3 -> 0
- net row5: track 366.1 -> 446.8 mm, vias 2 -> 3
- net row3: track 272.0 -> 335.7 mm, vias 0 -> 3
- net row4: track 331.8 -> 388.8 mm, vias 0 -> 3
- net row0: track 407.6 -> 352.7 mm, vias 4 -> 1
- net col16: track 180.7 -> 131.1 mm, vias 0 -> 2
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- removed copper zone on B.Cu, net +3V3
Other:
- board size 355.7 x 122.3 mm -> 355.7 x 134.5 mm
