File: keyboard.sch (KiCad schematic (older format))
At the start: 199 parts, among them J1 USB_B_Micro, J2 Conn_01x02, U1 NCP1117-3.3_SOT223, U2 W25Q128JVS, U3 RP2040, Y1 ABLS-12.000MHZ-B4-T

Commit message: add breakout, mini-DIN, and display headers; re-route
Parts:
- added C6, C7: 100n, Capacitor_SMD:C_0402_1005Metric, symbol Device:C_Small
- added C8: 1u, Capacitor_SMD:C_0402_1005Metric, symbol Device:C_Small
- added D88, D89, D90, D91: 1N4148W, Diode_SMD:D_0402_1005Metric, symbol Diode:1N4148W
- added J3: Mini-DIN-6, RP2040_minimal:MJD-006-FS, symbol MCU_RaspberryPi_RP2040:MDJ-006-FS
- added J4: Breakout, Connector_PinHeader_2.54mm:PinHeader_1x07_P2.54mm_Vertical, symbol Connector_Generic:Conn_01x07
- added J5: I2C_Display_Header, Connector_PinHeader_2.54mm:PinHeader_1x04_P2.54mm_Horizontal, symbol Connector_Generic:Conn_01x04
Connections:
- net GPIO10 is gone; now on net col4: U3.13 (GPIO10)
- net GPIO11 is gone; now on net col3: U3.14 (GPIO11)
- net GPIO12 is gone; now on net col2: U3.15 (GPIO12)
- net GPIO13 is gone; now on net col1: U3.16 (GPIO13)
- net GPIO14 is gone; now on net col0: U3.17 (GPIO14)
- net GPIO15 is gone; now on net col15: U3.18 (GPIO15)
- net +3V3: now also D90.2 (A)
- net GND: now also C6.2, C7.2, C8.2, J3.3, J4.7 (Pin_7), J5.1 (Pin_1)
- net VBUS: now also D88.1 (K), D89.1 (K), D91.1 (K), J5.3 (Pin_3); no longer J1.1 (VBUS)
- net col0: no longer U3.2 (GPIO0)
- net col1: no longer U3.3 (GPIO1)
- net col10: now also U3.3 (GPIO1); no longer U3.32 (GPIO21)
- net col11: now also U3.4 (GPIO2); no longer U3.31 (GPIO20)
- net col12: now also U3.5 (GPIO3); no longer U3.30 (GPIO19)
- net col13: now also U3.6 (GPIO4); no longer U3.29 (GPIO18)
- net col14: now also U3.7 (GPIO5); no longer U3.28 (GPIO17)
- net col15: no longer U3.41 (GPIO29_ADC3)
- net col16: now also U3.27 (GPIO16); no longer U3.39 (GPIO27_ADC1)
- net col17: now also U3.28 (GPIO17); no longer U3.36 (GPIO24)
- net col2: no longer U3.4 (GPIO2)
- net col3: no longer U3.5 (GPIO3)
- net col4: no longer U3.6 (GPIO4)
- net col5: now also U3.12 (GPIO9); no longer U3.7 (GPIO5)
- net col6: now also U3.11 (GPIO8); no longer U3.8 (GPIO6)
- net col8: now also U3.8 (GPIO6); no longer U3.11 (GPIO8)
- net col9: now also U3.2 (GPIO0); no longer U3.12 (GPIO9)
- net row0: now also U3.29 (GPIO18); no longer U3.35 (GPIO23)
- net row1: now also U3.30 (GPIO19); no longer U3.34 (GPIO22)
- net row2: now also U3.31 (GPIO20); no longer U3.37 (GPIO25)
- net row3: now also U3.32 (GPIO21); no longer U3.27 (GPIO16)
- net row4: now also U3.34 (GPIO22); no longer U3.38 (GPIO26_ADC0)
- net row5: now also U3.35 (GPIO23); no longer U3.40 (GPIO28_ADC2)
- net +1V1: now reaches U3.23 (DVDD)
- net +1V1: now also U3.45 (VREG_VOUT), U3.50 (DVDD), C6.1, C7.1, C8.1
- new net: D88.2 (A), J1.1 (VBUS)
- new net: D91.2 (A), J3.5
- new net: D89.2 (A), J4.5 (Pin_5)
- new net: D90.1 (K), J4.6 (Pin_6)
- new net GPIO24: J3.1, J4.1 (Pin_1), U3.36 (GPIO24)
- new net GPIO25: J3.6, J4.2 (Pin_2), U3.37 (GPIO25)
- new net GPIO26_ADC0: J3.8, J4.3 (Pin_3), U3.38 (GPIO26_ADC0)
- new net GPIO27_ADC1: J3.2, J4.4 (Pin_4), U3.39 (GPIO27_ADC1)
- new net I2C_SCL: J5.4 (Pin_4), U3.41 (GPIO29_ADC3)
- new net I2C_SDA: J5.2 (Pin_2), U3.40 (GPIO28_ADC2)
- no-connect marks 7 -> 4
